Commit message: Part 1: Complete barista robot with laser and diff drive

File: urdf/barista_robot_model.urdf (robot description, URDF)
Before this commit: robot barista_robot, 9 links, 8 joints
Links:
- added link laser_link; visual mesh filename=package://barista_robot_description/meshes/hokuyo_utm_30lx.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 scale=0.001 0.001 0.001
Joints:
- added joint laser_joint: type fixed, parent top_plate, child laser_link, origin xyz=0.05 0 0.05

Commit message: Checkpoint 7 Part 1: URDF robot with laser and diff drive plugin

File: urdf/barista_robot_model.urdf (robot description, URDF)
Before this commit: robot barista_robot, 10 links, 9 joints
Links:
- link standoff_1: geometry visual cylinder length=0.2 radius=0.01
- link standoff_2: geometry visual cylinder length=0.2 radius=0.01
- link standoff_3: geometry visual cylinder length=0.2 radius=0.01
- link standoff_4: geometry visual cylinder length=0.2 radius=0.01
